File: S2.1-Wrover-dev-pcb.kicad_pcb (KiCad board)
At the start: 2 copper layers, 99.1 x 50 mm, 28 parts, among them J1 USB_C_Receptacle_USB2.0, J2 Jack-DC, P1 CONN_02X13, P3 CONN_02X13, SW1 RESET, SW2 BOOT, U1 MCP1700-1202E_SOT23, U3 TPS2113APW, U4 TP4056

Commit message: Add Schottky btw. VBUS & TP4056 VCC
Parts:
- added D1: D_Schottky, Diode_SMD:D_SOD-123, F.Cu at (158.4, 90.4)
Connections:
- D2 pad 2: VBUS -> Net-(D1-Pad1)
- D3 pad 2: VBUS -> Net-(D1-Pad1)
- U4 pad 4: VBUS -> Net-(D1-Pad1)
- U4 pad 8: VBUS -> Net-(D1-Pad1)
Other:
- copper layers 2 -> 4
Changed lines of the file:
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@@
   (layers
     (0 "F.Cu" signal)
+    (1 "In1.Cu" signal)
+    (2 "In2.Cu" signal)
     (31 "B.Cu" signal)
     (32 "B.Adhes" user "B.Adhesive")
@@
       (layer "F.Mask" (type "Top Solder Mask") (color "Green") (thickness 0.01))
       (layer "F.Cu" (type "copper") (thickness 0.035))
-      (layer "dielectric 1" (type "core") (thickness 1.51) (material "FR4") (epsilon_r 4.5) (loss_tangent 0.02))
+      (layer "dielectric 1" (type "core") (thickness 0.48) (material "FR4") (epsilon_r 4.5) (loss_tangent 0.02))
+      (layer "In1.Cu" (type "copper") (thickness 0.035))
+      (layer "dielectric 2" (type "prepreg") (thickness 0.48) (material "FR4") (epsilon_r 4.5) (loss_tangent 0.02))
+      (layer "In2.Cu" (type "copper") (thickness 0.035))
+      (layer "dielectric 3" (type "core") (thickness 0.48) (material "FR4") (epsilon_r 4.5) (loss_tangent 0.02))
       (layer "B.Cu" (type "copper") (thickness 0.035))
-      (layer "B.Mask" (type "Bottom Solder Mask") (color "Green") (thickness 0.01))
+      (layer "B.Mask" (type "Bottom Solder Mask") (color "Red") (thickness 0.01))
       (layer "B.Paste" (type "Bottom Solder Paste"))
-      (layer "B.SilkS" (type "Bottom Silk Screen"))
+      (layer "B.SilkS" (type "Bottom Silk Screen") (color "White"))
       (copper_finish "None")
       (dielectric_constraints no)
@@
   (net 66 "unconnected-(P3-Pad26)")
   (net 67 "VIN")
+  (net 68 "Net-(D1-Pad1)")
   (footprint "Mounting_Holes:MountingHole_3-5mm" locked (layer "F.Cu")
     (at 191.76 117.33)
@@
     )
   )
+  (footprint "Diode_SMD:D_SOD-123" (layer "F.Cu")
+    (at 158.445 90.43 90)
+    (descr "SOD-123")
+    (tags "SOD-123")
+    (property "LCSC" "C8598")
+    (property "Sheetfile" "S2-Wrover-dev-pcb.kicad_sch")
+    (property "Sheetname" "")
+    (attr smd)
+    (fp_text reference "D1" (at 0 -2 90) (layer "F.SilkS")
+      (effects (font (size 1 1) (thickness 0.15)))
+    )
+    (fp_text value "D_Schottky" (at 0 2.1 90) (layer "F.Fab")
+      (effects (font (size 1 1) (thickness 0.15)))
+    )
+    (fp_text user "${REFERENCE}" (at 0 -2 90) (layer "F.Fab")
+      (effects (font (size 1 1) (thickness 0.15)))
+    )
+    (fp_line (start -2.25 -1) (end -2.25 1) (layer "F.SilkS") (width 0.12))
+    (fp_line (start -2.25 1) (end 1.65 1) (layer "F.SilkS") (width 0.12))
+    (fp_line (start -2.25 -1) (end 1.65 -1) (layer "F.SilkS") (width 0.12))
+    (fp_line (start 2.35 1.15) (end -2.35 1.15) (layer "F.CrtYd") (width 0.05))
+    (fp_line (start -2.35 -1.15) (end 2.35 -1.15) (layer "F.CrtYd") (width 0.05))
+    (fp_line (start -2.35 -1.15) (end -2.35 1.15) (layer "F.CrtYd") (width 0.05))
+    (fp_line (start 2.35 -1.15) (end 2.35 1.15) (layer "F.CrtYd") (width 0.05))
+    (fp_line (start 1.4 -0.9) (end 1.4 0.9) (layer "F.Fab") (width 0.1))
+    (fp_line (start 0.25 0.4) (end -0.35 0) (layer "F.Fab") (width 0.1))
+    (fp_line (start -0.75 0) (end -0.35 0) (layer "F.Fab") (width 0.1))
+    (fp_line (start 0.25 -0.4) (end 0.25 0.4) (layer "F.Fab") (width 0.1))
+    (fp_line (start -1.4 0.9) (end -1.4 -0.9) (layer "F.Fab") (width 0.1))
+    (fp_line (start 1.4 0.9) (end -1.4 0.9) (layer "F.Fab") (width 0.1))
+    (fp_line (start 0.25 0) (end 0.75 0) (layer "F.Fab") (width 0.1))
+    (fp_line (start -0.35 0) (end -0.35 0.55) (layer "F.Fab") (width 0.1))
+    (fp_line (start -1.4 -0.9) (end 1.4 -0.9) (layer "F.Fab") (width 0.1))
+    (fp_line (start -0.35 0) (end -0.35 -0.55) (layer "F.Fab") (width 0.1))
+    (fp_line (start -0.35 0) (end 0.25 -0.4) (layer "F.Fab") (width 0.1))
+    (pad "1" smd rect (at -1.65 0 90) (size 0.9 1.2) (layers "F.Cu" "F.Paste" "F.Mask")
+      (net 68 "Net-(D1-Pad1)") (pinfunction "K") (pintype "passive"))
+    (pad "2" smd rect (at 1.65 0 90) (size 0.9 1.2) (layers "F.Cu" "F.Paste" "F.Mask")
+      (net 8 "VBUS") (pinfunction "A") (pintype "passive"))
+    (model "${KICAD6_3DMODEL_DIR}/Diode_SMD.3dshapes/D_SOD-123.wrl"
+      (offset (xyz 0 0 0))
+      (scale (xyz 1 1 1))
+      (rotate (xyz 0 0 0))
+    )
+  )
   (footprint "LED_SMD:LED_0805_2012Metric" (layer "F.Cu")
     (at 183.2075 107.205)
@@
       (net 18 "Net-(D3-Pad1)") (pinfunction "K") (pintype "passive"))
     (pad "2" smd roundrect (at 0.9375 0) (size 0.975 1.4) (layers "F.Cu" "F.Paste" "F.Mask") (roundrect_rratio 0.25)
-      (net 8 "VBUS") (pinfunction "A") (pintype "passive"))
+      (net 68 "Net-(D1-Pad1)") (pinfunction "A") (pintype "passive"))
     (model "${KICAD6_3DMODEL_DIR}/LED_SMD.3dshapes/LED_0805_2012Metric.wrl"
       (offset (xyz 0 0 0))
@@
       (net 1 "GND") (pinfunction "GND") (pintype "power_in"))
     (pad "4" smd rect (at -2.7 1.905 90) (size 1.5 0.65) (layers "F.Cu" "F.Paste" "F.Mask")
-      (net 8 "VBUS") (pinfunction "VCC") (pintype "power_in"))
+      (net 68 "Net-(D1-Pad1)") (pinfunction "VCC") (pintype "power_in"))
     (pad "5" smd rect (at 2.7 1.905 90) (size 1.5 0.65) (layers "F.Cu" "F.Paste" "F.Mask")
       (net 9 "BAT+") (pinfunction "BAT") (pintype "power_out"))
@@
       (net 16 "Net-(R3-Pad2)") (pinfunction "~{CHRG}") (pintype "open_collector"))
     (pad "8" smd rect (at 2.7 -1.905 90) (size 1.5 0.65) (layers "F.Cu" "F.Paste" "F.Mask")
-      (net 8 "VBUS") (pinfunction "CE") (pintype "input"))
+      (net 68 "Net-(D1-Pad1)") (pinfunction "CE") (pintype "input"))
     (pad "9" smd rect (at 0 0 90) (size 2.7 3.6) (layers "F.Cu" "F.Paste" "F.Mask")
       (net 17 "unconnected-(U4-Pad9)") (pinfunction "PP") (pintype "input+no_connect"))
@@
       (net 19 "Net-(D2-Pad1)") (pinfunction "K") (pintype "passive"))
     (pad "2" smd roundrect (at 0.9375 0 180) (size 0.975 1.4) (layers "F.Cu" "F.Paste" "F.Mask") (roundrect_rratio 0.25)
-      (net 8 "VBUS") (pinfunction "A") (pintype "passive"))
+      (net 68 "Net-(D1-Pad1)") (pinfunction "A") (pintype "passive"))
     (model "${KICAD6_3DMODEL_DIR}/LED_SMD.3dshapes/LED_0805_2012Metric.wrl"
       (offset (xyz 0 0 0))
