File: PMIC-tester/S2-PMIC-dev-pcb.kicad_pcb (KiCad board)
At the start: 2 copper layers, 99.1 x 50 mm, 29 parts, among them J1 USB_C_Receptacle_USB2.0, P1 CONN_02X13, P3 CONN_02X13, SW1 RESET, SW2 BOOT, U1 MCP1700-1202E_SOT23, U2 ESP32-S2-WROVER, U3 TPS65185RGZR

Commit message: min. clearance 0,18mm
Routing:
- net Net-(C2-Pad1): track 18.7 -> 28.7 mm
Changed lines of the file:
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@@
     (property "Sheetfile" "S2-PMIC-dev-pcb.kicad_sch")
     (property "Sheetname" "")
+    (clearance 0.15)
     (attr through_hole)
     (fp_text reference "U3" (at -5.125 -3.65) (layer "F.SilkS")
@@
   (segment (start 152.845 82.305) (end 179.045 82.305) (width 0.2) (layer "B.Cu") (net 12))
   (segment (start 181.645 80.255) (end 181.995 80.605) (width 0.4) (layer "F.Cu") (net 13))
+  (segment (start 178.37 78.93) (end 176.97 80.33) (width 0.4) (layer "F.Cu") (net 13))
   (segment (start 183.795 80.605) (end 184.1 80.3) (width 0.4) (layer "F.Cu") (net 13))
+  (segment (start 176.97 80.33) (end 172.225 80.33) (width 0.4) (layer "F.Cu") (net 13))
+  (segment (start 181.645 78.93) (end 178.37 78.93) (width 0.4) (layer "F.Cu") (net 13))
   (segment (start 189.425 84.975) (end 190.905 86.455) (width 0.4) (layer "F.Cu") (net 13))
   (segment (start 181.645 78.93) (end 187.255 78.93) (width 0.4) (layer "F.Cu") (net 13))

Commit message: DRC
Connections:
- P3 pad 22: unconnected-(P3-Pad22) -> /IO36
- P3 pad 24: unconnected-(P3-Pad24) -> /IO37
Routing:
- net /IO37: track 0.00 -> 19.0 mm
- net /IO36: track 0.00 -> 17.1 mm
- net /+22V: track 36.0 -> 35.1 mm
- net /-15V: track 48.0 -> 47.3 mm
Other:
- board text added: "3.3V"
- board text added: "GND"
- board text added: "IO13"
- board text added: "IO14"
- board text added: "IO15"
- board text added: "IO16"
- board text added: "IO17"
- board text added: "IO18"
- board text added: "IO21"
- board text added: "IO33"
- board text added: "IO34"
- board text added: "IO35"
- board text added: "IO36"
- board text added: "IO37"
- board text added: "IO38"
- board text added: "IO39"
- board text added: "IO40"
- board text added: "IO41"
- board text added: "IO42"
- board text added: "IO45"
- board text added: "RX"
- board text added: "TX"
- board text removed: "3.3 | 15"
- board text removed: "3.3 | 16"
- board text removed: "38 | x"
- board text removed: "39 | 35"
- board text removed: "40 | 34"
- board text removed: "41 | 33"
- board text removed: "42 | 21"
- board text removed: "45 | 18"
- board text removed: "GND | 13"
- board text removed: "GND | 14"
- board text removed: "I46 | 17"
- board text removed: "RX | 37"
- board text removed: "TX | x"

Commit message: I2C pullups
Parts:
- added R5: 2k2, Resistor_SMD:R_0603_1608Metric, F.Cu at (146.6, 92.7)
- added R8: 2k2, Resistor_SMD:R_0603_1608Metric, F.Cu at (146.6, 96.3)
Routing:
- net /3.3V: track 197.4 -> 209.3 mm, vias 5 -> 7
- net /SDA: track 46.1 -> 49.0 mm
- net /SCL: track 46.8 -> 49.5 mm
